File: plottercard.kicad_sch (KiCad schematic)
At the start: 70 parts, among them J10 SLTpad, J11 SLTpad, J12 SLTpad, J13 SLTpad, J2 SLTpad, J3 SLTpad, J4 SLTpad, J5 SLTpad, J6 SLTpad, J7 SLTpad, J8 SLTpad, J9 SLTpad, U20 74LS05, U21 LD1117S50TR_SOT223, U6 74LS07, X1 Conn_01x09_Socket, X2 Conn_01x09_Socket, X3 Conn_01x09_Socket, X4 Conn_01x09_Socket

Commit message: Up to date KiCad design files
matching the gerbers and drill files
Parts:
- removed B10, B11, B12, B13, B2, B3, B4, B5, B6, B7, B8, B9, D10, D11, D12, D13, D2, D3, D4, D5, D6, D7, D8, D9, G10, G11, G12, G13, G2, G3, G4, G5, G6, G7, G8, G9, J10, J11, J12, J13, J2, J3, J4, J5, J6, J7, J8, J9: SLTpad, Library.carl:SLTpad, symbol carl:SLTpad
- added J14: EdgeConnectorSingle, IBM:PlugConnector, symbol IBMCards:EdgeConnectorSingle
- added J15: EdgeConnectorSingle2, IBM:PlugConnector2, symbol IBMCards:EdgeConnectorSingle2
- added J16: Conn_01x02_Pin, Connector_PinHeader_2.54mm:PinHeader_1x02_P2.54mm_Vertical, symbol Connector:Conn_01x02_Pin
- renumbered X4 to X3, X3 to X4
Connections:
- net +12V: now also J15.G02
- net GND: now also X4.9 (Pin_9), J14.D08, J15.J08, J16.2 (Pin_2); no longer X3.9 (Pin_9)
- net at C27.1, C6.1, C8.1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: now also X3.9 (Pin_9); no longer X4.9 (Pin_9)
- net at X1.5 (Pin_5): now also J14.B03
- net at R11.2, R12.1: now also J14.B08
- net at U20.3: now also X3.2 (Pin_2); no longer X4.2 (Pin_2)
- net at U20.4: now also J14.B10
- net at R1.2, U6.2: now also J15.J05
- net at R4.2, U6.10: now also J15.J04
- net at X4.1 (Pin_1): no longer U20.1
- net at X4.5 (Pin_5): now also J14.D09
- net at X4.6 (Pin_6): now also J14.D07, J14.D11
- net at X1.1 (Pin_1): now also J15.J12
- net at X1.2 (Pin_2): now also J15.J10
- net at X1.3 (Pin_3): now also J15.J13
- net at X1.4 (Pin_4): now also J14.D12
- net at X1.6 (Pin_6): now also J14.D10
- net at X1.7 (Pin_7): now also J14.D02
- net at X1.8 (Pin_8): now also J14.D13
- net at X1.9 (Pin_9): now also J14.D06
- net at U20.6: now also J14.B04
- net at U20.2: now also J14.B09
- net at R3.2, U6.6: now also J15.G05
- net at R2.2, U6.4: now also J15.J02
- net at R5.2, U6.12: now also J14.D04
- net at R6.2, U6.8: now also J14.D05
- net at X2.7 (Pin_7): now also J14.B02
- net at X3.1 (Pin_1): now also U20.1
- net at X3.8 (Pin_8): now also J16.1 (Pin_1)
- net at U20.8: now also J14.B05
- no-connect marks 33 -> 32
Other:
- note added: "Substitute card for IBM 5806223 Implements controller logic for IBM 1627 plotter when attached to an IBM 1130 computing system"
- note added: "jumper installed on J1 if 1627 model 2 or Calcomp 563 is attached"
- note added: "model1"
- moved on the sheet: C26, C27, C6, C8, R1, R11, R12, R13, R2, R3, R4, R5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
